File: KiCAD/Pro-Controller-X/StickLeft.kicad_pcb (KiCad board)
At the start: 2 copper layers, 32 x 34 mm, 2 parts, among them J1 Conn_01x05_Pin

Commit message: Final Revision - Boards Ordered
Other:
- board text added: "Lego_Rocket"
- board text added: "U1"
Changed lines of the file:
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@@
       (drillshape 0)
       (scaleselection 1)
-      (outputdirectory "../../Outputs/")
+      (outputdirectory "../../Outputs/StickLeft/")
     )
   )
@@
         (effects (font (size 1 1) (thickness 0.15)) (justify mirror))
     )
-    (fp_text user "${REFERENCE}" (at -1.8 0.4 90) (layer "F.Fab")
+    (fp_text user "${REFERENCE}" (at 0.06 -1.658 90) (layer "F.Fab")
         (effects (font (size 1.27 1.27) (thickness 0.254)))
     )
@@
     (fp_line (start 13.7 1.4) (end 12.959133 2.104768)
       (stroke (width 0.12) (type default)) (layer "Edge.Cuts"))
-    (fp_arc (start -17.996881 2.405549) (mid -14.574017 -7.204322) (end -5.91618 -12.599455)
+    (fp_arc (start -17.996881 2.405549) (mid -14.574017 -7.204321) (end -5.91618 -12.599455)
       (stroke (width 0.12) (type default)) (layer "Edge.Cuts"))
     (fp_arc (start -10.400305 15.500567) (mid -13.063389 13.705077) (end -15.299999 11.4)
@@
       (net 3 "GND") (pinfunction "MH2") (pintype "input"))
   )
+  (gr_text "Lego_Rocket" (at 150 103.5) (layer "B.SilkS")
+    (effects (font (size 1.5 1.5) (thickness 0.3) bold) (justify left bottom mirror))
+  )
+  (gr_text "U1" (at 140 106.5 90) (layer "B.SilkS")
+    (effects (font (size 1.27 1.27) (thickness 0.254)) (justify mirror))
+  )
   (segment (start 147.54 105.19) (end 145.62 107.11) (width 0.5) (layer "B.Cu") (net 1))
