File: KiCAD/Pro-Controller-X/StickRight.kicad_pcb (KiCad board)
At the start: 2 copper layers, 32.8 x 34 mm, 2 parts, among them J1 Conn_01x05_Pin

Commit message: Joystick Boards done
Parts:
- J1: moved to F.Cu
- moved J1 10.2 mm to (147.3, 96.6)
Connections:
- J1 pad 1: unconnected-(J1-Pin_1-Pad1) -> Net-(J1-Pin_1)
- J1 pad 2: unconnected-(J1-Pin_2-Pad2) -> Net-(J1-Pin_2)
- J1 pad 3: unconnected-(J1-Pin_3-Pad3) -> Net-(J1-Pin_3)
- J1 pad 4: unconnected-(J1-Pin_4-Pad4) -> GND
- J1 pad 5: unconnected-(J1-Pin_5-Pad5) -> Net-(J1-Pin_5)
- U1 pad A1: unconnected-(U1-PadA1) -> GND
- U1 pad A11: unconnected-(U1-PadA11) -> Net-(J1-Pin_1)
- U1 pad A12: unconnected-(U1-PadA12) -> Net-(J1-Pin_3)
- U1 pad A13: unconnected-(U1-PadA13) -> GND
- U1 pad B1: unconnected-(U1-PadB1) -> Net-(J1-Pin_5)
- U1 pad B11: unconnected-(U1-PadB11) -> Net-(J1-Pin_1)
- U1 pad B12: unconnected-(U1-PadB12) -> Net-(J1-Pin_2)
- U1 pad B13: unconnected-(U1-PadB13) -> GND
- U1 pad MH1: unconnected-(U1-PadMH1) -> GND
- U1 pad MH2: unconnected-(U1-PadMH2) -> GND
Routing:
- net Net-(J1-Pin_1): track 0.00 -> 32.4 mm
- net Net-(J1-Pin_5): track 0.00 -> 23.1 mm
- net Net-(J1-Pin_2): track 0.00 -> 19.2 mm
- net Net-(J1-Pin_3): track 0.00 -> 8.99 mm
- net GND: vias 0 -> 14
- added copper zone on B.Cu, net GND
- added copper zone on F.Cu, net GND
