File: KiCAD/Pro-Controller-X/StickRight.kicad_pcb (KiCad board)
At the start: 2 copper layers, 32.8 x 34 mm, 2 parts, among them J1 Conn_01x05_Pin

Commit message: Final Revision - Boards Ordered
Other:
- board text added: "Lego_Rocket"
Changed lines of the file:
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@@
     (property "Sheetname" "")
     (attr smd)
-    (fp_text reference "U1" (at 0 0.5 unlocked) (layer "B.SilkS")
+    (fp_text reference "U1" (at -2.7325 -1.467 unlocked) (layer "B.SilkS")
         (effects (font (size 1 1) (thickness 0.15)) (justify mirror))
     )
@@
         (effects (font (size 1 1) (thickness 0.15)) (justify mirror))
     )
-    (fp_text user "${REFERENCE}" (at 1.0125 0.351 90) (layer "F.Fab")
+    (fp_text user "${REFERENCE}" (at 2.7675 -1.967 90) (layer "F.Fab")
         (effects (font (size 1.27 1.27) (thickness 0.254)))
     )
@@
       (net 5 "GND") (pinfunction "MH2") (pintype "input"))
   )
+  (gr_text "Lego_Rocket" (at 143.5 81.5) (layer "B.SilkS")
+    (effects (font (size 1.5 1.5) (thickness 0.3) bold) (justify left bottom mirror))
+  )
   (segment (start 137.04 81.75) (end 146.065 81.75) (width 0.5) (layer "B.Cu") (net 1))
