File: KiCAD/Pro-Controller-X/Pro-Controller-X.kicad_sch (KiCad schematic)
At the start: 77 parts, among them J2 USB_C_Receptacle_USB2.0, Q1 2N7002, Q2 2N7002, Q3 2N7002, Q4 2N7002, Q5 2N7002, Q6 2N7002, Q7 2N7002, Q8 2N7002, U1 TP4056

Commit message: Rough Antenna outline for placement
Parts:
- added U6: ~, ProControllerX:MCU8BitDo, symbol ProControllerX:MCU8BitDo
Changed lines of the file:
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@@
+    )
+  )
+  (symbol (lib_id "ProControllerX:MCU8BitDo") (at 486.41 67.31 0) (unit 1)
+    (in_bom yes) (on_board yes) (dnp no) (fields_autoplaced)
+    (property "Reference" "U6" (at 511.81 140.97 0)
+      (effects (font (size 1.27 1.27)) (justify left))
+    )
+    (property "Value" "~" (at 485.14 113.03 0)
+      (effects (font (size 1.27 1.27)))
+    )
+    (property "Footprint" "ProControllerX:MCU8BitDo" (at 485.14 113.03 0)
+      (effects (font (size 1.27 1.27)) hide)
+    )
+    (property "Datasheet" "" (at 485.14 113.03 0)
+      (effects (font (size 1.27 1.27)) hide)
+    )
+    (pin "1")
+    (pin "10")
+    (pin "11")
+    (pin "12")
+    (pin "13")
+    (pin "14")
+    (pin "15")
+    (pin "16")
+    (pin "17")
+    (pin "18")
+    (pin "19")
+    (pin "2")
+    (pin "20")
+    (pin "21")
+    (pin "22")
+    (pin "23")
+    (pin "24")
+    (pin "25")
+    (pin "26")
+    (pin "27")
+    (pin "28")
+    (pin "29")
+    (pin "3")
+    (pin "30")
+    (pin "31")
+    (pin "32")
+    (pin "33")
+    (pin "34")
+    (pin "35")
+    (pin "36")
+    (pin "37")
+    (pin "38")
+    (pin "39")
+    (pin "4")
+    (pin "40")
+    (pin "41")
+    (pin "42")
+    (pin "5")
+    (pin "6")
+    (pin "7")
+    (pin "8")
+    (pin "9")
+    (instances
+      (project "Pro-Controller-X"
+        (path "/40a7657d-c4d7-4ebc-b606-0c6932d6f433"
+          (reference "U6") (unit 1)
+        )
+      )
     )
   )

Commit message: Joystick Boards done
Parts:
- D1, D2, D3, D4, D5: footprint (none) -> LED_SMD:LED_0603_1608Metric
Changed lines of the file:
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@@
       (effects (font (size 1.27 1.27)))
     )
-    (property "Footprint" "" (at 139.7 313.69 0)
+    (property "Footprint" "LED_SMD:LED_0603_1608Metric" (at 139.7 313.69 0)
       (effects (font (size 1.27 1.27)) hide)
     )
@@
       (effects (font (size 1.27 1.27)))
     )
-    (property "Footprint" "" (at 139.7 303.53 0)
+    (property "Footprint" "LED_SMD:LED_0603_1608Metric" (at 139.7 303.53 0)
       (effects (font (size 1.27 1.27)) hide)
     )
@@
       (effects (font (size 1.27 1.27)))
     )
-    (property "Footprint" "" (at 130.81 267.97 0)
+    (property "Footprint" "LED_SMD:LED_0603_1608Metric" (at 130.81 267.97 0)
       (effects (font (size 1.27 1.27)) hide)
     )
@@
       (effects (font (size 1.27 1.27)))
     )
-    (property "Footprint" "" (at 139.7 293.37 0)
+    (property "Footprint" "LED_SMD:LED_0603_1608Metric" (at 139.7 293.37 0)
       (effects (font (size 1.27 1.27)) hide)
     )
@@
       (effects (font (size 1.27 1.27)))
     )
-    (property "Footprint" "" (at 139.7 283.21 0)
-      (effects (font (size 1.27 1.27)) hide)
-    )
+    (property "Footprint" "LED_SMD:LED_0603_1608Metric" (at 139.7 283.21 0)
+      (effects (font (size 1.27 1.27)) hide)
+    )

Commit message: Most MCU Pins Mapped
Parts:
- added C18, C19, C20, C21: C, Capacitor_SMD:C_0402_1005Metric_Pad0.74x0.62mm_HandSolder, symbol Device:C
- added R34, R35, R36, R37: R_US, Resistor_SMD:R_0402_1005Metric_Pad0.72x0.64mm_HandSolder, symbol Device:R_US
Connections:
- net RDIV-BC is gone; now on net V_DIV: C4.2, R1.1, R2.2
- net CHRG: now also U6.42 (Tp4056), R35.1
- net GND: now also C16.1, C17.2, R22.2, R33.1, U6.1 (GND), C18.2, C19.2, C20.2, C21.2, R36.2
- net VCC: now also R14.2
- net VDD: now also C16.2, C17.1, C6.1, Q1.3 (D), R12.1, R31.2, R32.2, U3.5, U5.12, U5.5, U5.8, U6.2 (V+), R35.2; no longer C3.1, D12.2 (A), D13.1 (K), Q2.2 (S), R16.1, R8.1, U1.5 (BAT)
- net at U5.1: now also R33.2
- net at D4.2 (A): now also U6.17 (P4_LED)
- net RMBL: now reaches R29.2
- net RMBL: now also U6.11 (Rmbl)
- net at D3.2 (A): now also U6.18 (P3_LED)
- net BTN_A: now reaches U2.1 (A)
- net BTN_A: now also U6.15 (Btn_A)
- net BTN_LEFT: now reaches U2.10 (Left)
- net BTN_LEFT: now also U6.28 (Btn_Left)
- net BTN_DOWN: now reaches U2.11 (Down)
- net BTN_DOWN: now also U6.29 (Btn_Down)
- net BTN_RIGHT: now reaches U2.12 (Right)
- net BTN_RIGHT: now also U6.27 (Btn_Right)
- net BTN_L: now reaches U2.13 (L)
- net BTN_L: now also U6.32 (Btn_L)
- net BTN_ZL: now reaches U2.14 (ZL)
- net BTN_ZL: now also U6.10 (Btn_ZL)
- net BTN_R: now reaches U2.15 (R)
- net BTN_R: now also U6.9 (Btn_R)
- net BTN_ZR: now reaches U2.16 (ZR)
- net BTN_ZR: now also U6.35 (Btn_ZR)
- net SYNC: now reaches U2.17 (Sync)
- net SYNC: now also U6.8 (Btn_Sync)
- net BTN_B: now reaches U2.2 (B)
- net BTN_B: now also U6.16 (Btn_B)
- net BTN_X: now reaches U2.3 (X)
- net BTN_X: now also R34.1
- net Y1: now reaches U2.39 (Y1)
- net Y1: now also U6.38 (RStick*), C20.1
- net BTN_Y: now reaches U2.4 (Y)
- net BTN_Y: now also U6.6 (Btn_Y)
- net VDC: now reaches U2.40 (V+)
- net VDC: now also C5.1, Q1.2 (S)
- net X1: now reaches U2.41 (X1)
- net X1: now also U6.37 (RStick*), C21.1
- net BTN1: now reaches U2.43 (Btn1)
- net BTN1: now also U6.12 (RStick*)
- net Y2: now reaches U2.44 (Y2)
- net Y2: now also U6.40 (LStick*), C18.1
- net X2: now reaches U2.45 (X2)
- net X2: now also U6.39 (LStick*), C19.1
- net BTN2: now reaches U2.46 (Btn2)
- net BTN2: now also U6.3 (LStick*)
- net BTN_PLU: now reaches U2.5 (+)
- net BTN_PLU: now also U6.26 (Btn_Plus)
- net BTN_MIN: now reaches U2.6 (-)
- net BTN_MIN: now also U6.34 (Btn_Minus)
- net BTN_STR: now reaches U2.7 (Home)
- net BTN_STR: now also R37.1
- net BTN_HME: now reaches U2.8 (Pwr)
- net BTN_HME: now also Q4.1 (G)
- net BTN_UP: now reaches U2.9 (Up)
- net BTN_UP: now also U6.41 (Btn_Up)
- net at D5.2 (A): now also U6.33 (LED_Sync)
- net DIV: now reaches C9.1, R10.1, R9.2
- net DIV: now also U6.36 (Ctr_Circuit)
- net at D2.2 (A): now also U6.13 (P2_LED)
- net D-: now reaches R24.2
- net D+: now reaches R23.2
- net at D1.2 (A): now also U6.14 (P1_LED)
- net at R6.2: now also R36.1
- net BTN_CR: now reaches U6.19 (Ctr_Circuit)
- net BTN_CR: now also Q4.3 (D)
- net CTR_CR: now reaches U6.25 (Ctr_Circuit)
- net CTR_CR: now also R13.2
- net V_DIV: now reaches U6.30 (Volt_Div)
- net at U6.31 (Btn_Star): now also R37.2
- net at U6.7 (Btn_X): now also R34.2
- new net V_BATT: C3.1, D12.2 (A), D13.1 (K), Q2.2 (S), R16.1, R8.1, U1.5 (BAT)
Other:
- moved on the sheet: C11, C16, C17, C3, C5, D1, D13, D2, D3, D4, D5, Q1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

Commit message: First rough routing complete
Parts:
- added J2: CONN_02PTH2, 1X02_BIG, symbol SparkFun-Connectors:CONN_02PTH2
- added R38, R39, R40, R41: R_US, Resistor_SMD:R_1206_3216Metric_Pad1.30x1.75mm_HandSolder, symbol Device:R_US
- C11: footprint Capacitor_SMD:C_0805_2012Metric_Pad1.18x1.45mm_HandSolder -> Capacitor_SMD:C_0402_1005Metric_Pad0.74x0.62mm_HandSolder
- C16, C17, C9: footprint Capacitor_SMD:C_0603_1608Metric -> Capacitor_SMD:C_0402_1005Metric_Pad0.74x0.62mm_HandSolder
- Q2, Q4, Q5: footprint Package_TO_SOT_SMD:SuperSOT-3 -> Package_TO_SOT_SMD:SOT-23
Connections:
- net D+: now also U6.21 (D+)
- net D-: now also U6.20 (D-)
- net GND: now also R39.2, R41.2; no longer U2.42 (Gnd)
- net VDC: now also R38.2, R40.2; no longer U2.40 (V+)
- net at C7.1, Q2.3 (D), U3.1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: now also R9.1, U4.3
- net i2c-: now reaches R32.1, U5.13 (i2c+*)
- net i2c-: now also U6.24 (i2c-*)
- net i2c+: now reaches R31.1, U5.14 (i2c-*)
- net i2c+: now also U6.23 (i2c+*)
- net USB-: now reaches D8.1 (K), J2.A7 (D-), J2.B7 (D-), R24.1
- net USB+: now reaches D7.2 (A), J2.A6 (D+), J2.B6 (D+), R23.1
- net RMBL-: now reaches C14.1, D10.1 (K), D9.2 (A), R30.1
- net RMBL-: now also J2.2
- net RMBL+: now reaches C15.2, D10.2 (A), D11.1 (K)
- net RMBL+: now also J2.1
- net at U6.4 (ANT2): now also U6.5 (ANT1)
- new net: R38.1, U2.40 (V+)
- new net: R39.1, U2.42 (Gnd)
- new net: R40.1, U2.47 (V+)
- new net: R41.1, U2.48 (Gnd)
