File: KiCAD/Pro-Controller-X/Pro-Controller-X.kicad_sch (KiCad schematic)
At the start: 95 parts, among them J2 CONN_02PTH2, J2 USB_C_Receptacle_USB2.0, J4 CONN_04, Q1 2N7002, Q2 2N7002, Q3 2N7002, Q4 2N7002, Q5 2N7002, Q6 2N7002, Q7 2N7002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

Commit message: Added Silkscreen Decoration
Parts:
- added REF3: LogoRef, ProControllerX:ProControllerLogo, symbol DSBB:LogoRef
Changed lines of the file:
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@@
+    )
+  )
+  (symbol (lib_id "DSBB:LogoRef") (at 448.31 273.05 0) (unit 1)
+    (in_bom yes) (on_board yes) (dnp no) (fields_autoplaced)
+    (property "Reference" "REF3" (at 458.47 272.415 0)
+      (effects (font (size 1.27 1.27)) (justify left))
+    )
+    (property "Value" "LogoRef" (at 458.47 274.955 0)
+      (effects (font (size 1.27 1.27)) (justify left))
+    )
+    (property "Footprint" "ProControllerX:ProControllerLogo" (at 448.31 273.05 0)
+      (effects (font (size 1.27 1.27)) hide)
+    )
+    (property "Datasheet" "" (at 448.31 273.05 0)
+      (effects (font (size 1.27 1.27)) hide)
+    )
+    (instances
+      (project "Pro-Controller-X"
+        (path "/40a7657d-c4d7-4ebc-b606-0c6932d6f433"
+          (reference "REF3") (unit 1)
+        )
+      )
     )
   )
